File: airspeed_v2/airspeed_v2.kicad_sch (KiCad schematic)
At the start: 20 parts, among them J1 Conn_01x04_Pin, J3 Conn_01x02_Pin, U1 XGZP6897D, U2 MPU-9250, U3 SHT4x, U4 MS5611-01BA, U5 XGZP6897D, U6 BME280

Commit message: airspeed v2
Parts:
- removed J1: Conn_01x04_Pin, Connector_PinHeader_2.54mm:PinHeader_1x04_P2.54mm_Vertical, symbol Connector:Conn_01x04_Pin
- removed J3: Conn_01x02_Pin, Connector_PinHeader_2.54mm:PinHeader_1x02_P2.54mm_Vertical, symbol Connector:Conn_01x02_Pin
- removed U4: MS5611-01BA, Package_LGA:LGA-8_3x5mm_P1.25mm, symbol Diff_Pressure:MS5611-01BA
- added C6: C, Capacitor_SMD:C_0805_2012Metric, symbol Device:C
- added C7, C8: C, symbol Device:C
- added C9: 0.1pF, Capacitor_Tantalum_SMD:CP_EIA-3216-18_Kemet-A, symbol Device:C
- added J1: Header, Connector_PinHeader_2.54mm:PinHeader_1x06_P2.54mm_Vertical, symbol Connector:Conn_01x06_Pin
- added J2: GPS, Connector_JST:JST_SH_SM06B-SRSS-TB_1x06-1MP_P1.00mm_Horizontal, symbol Connector:Conn_01x06_Pin
- added J3: GPS, Connector_PinHeader_1.27mm:PinHeader_1x06_P1.27mm_Vertical, symbol Connector:Conn_01x06_Pin
- added J4: ScreenIO, Connector_PinHeader_1.27mm:PinHeader_1x08_P1.27mm_Vertical, symbol Connector:Conn_01x08_Pin
- added JP1, JP2: 0x76 | 0x77, Jumper:SolderJumper-3_P2.0mm_Open_TrianglePad1.0x1.5mm, symbol Jumper:SolderJumper_3_Open
- added R4, R5, R6, R7: 10k, Resistor_SMD:R_0805_2012Metric, symbol Device:R
- added U8: BMP280, Package_LGA:Bosch_LGA-8_2x2.5mm_P0.65mm_ClockwisePinNumbering, symbol Diff_Pressure:BMP280
Connections:
- net 3v3 is gone; now on net +3V3: C1.1, C2.1, C3.1, C4.1, C5.1, R1.1, R2.1, U1.2 (VDD), U2.13 (VDD), U3.3 (VDD), U5.2 (VDD), U6.6 (VDDIO), U6.8 (VDD)
- net GND: now also U2.20 (RESV_GND), C6.2, C7.2, C8.2, C9.2, J1.2 (Pin_2), J2.3 (Pin_3), J3.3 (Pin_3), J4.3 (Pin_3), JP1.3 (B), JP2.1 (A), R6.2, U8.1 (GND), U8.7 (GND)
- net SCL: now also J1.4 (Pin_4), J2.5 (Pin_5), J3.5 (Pin_5), J4.5 (Pin_5)
- net SCL2: now also J1.6 (Pin_6), J4.8 (Pin_8), R4.2, U8.4 (SCK)
- net SDA: now also J1.3 (Pin_3), J2.6 (Pin_6), J3.6 (Pin_6), J4.6 (Pin_6)
- net SDA2: now also J1.5 (Pin_5), J4.7 (Pin_7), R5.2, U8.3 (SDI)
- net at R3.1: now also U2.11 (FSYNC); no longer U6.5 (SDO)
- net +3V3: now reaches U2.1 (RESV_VDDIO)
- net +3V3: now also U2.8 (VDDIO), U6.2 (CSB), C6.1, C7.1, C8.1, J1.1 (Pin_1), JP1.1 (A), JP2.3 (B), R4.1, R5.1, R7.1, U8.6 (VDDIO), U8.8 (VDD)
- net at U2.10 (REGOUT): now also C9.1
- net at U2.22 (~{CS}): now also R7.2
- net at U2.9 (AD0/MISO): now also R6.1
- new net: JP2.2 (C), U8.5 (SDO)
- new net: JP1.2 (C), U6.5 (SDO)
- new net 5V: J2.4 (Pin_4), J3.4 (Pin_4), J4.4 (Pin_4)
- new net Rx: J2.1 (Pin_1), J3.1 (Pin_1), J4.1 (Pin_1)
- new net Tx: J2.2 (Pin_2), J3.2 (Pin_2), J4.2 (Pin_2)
- no-connect marks 13 -> 4
Other:
- note added: "BMP280 Address: - 0x77 when connected to 3v3 - 0x76 when connected to GND"
- company: (none) -> velometa.com
- title: (none) -> Airspeed
- moved on the sheet: C1, C2, C3, C4, C5, H1, H2, H3, H4, R1, R2, U1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
