File: airspeed_v3/airspeed.kicad_pcb (KiCad board)
At the start: 2 copper layers, 40 x 40 mm, 22 parts, among them J1 Header, J2 GPS, J3 GPS, J4 ScreenIO, U1 XGZP6897D, U3 SHT4x, U5 XGZP6897D, U6 BME280, U8 BMP280

Commit message: complete airspeed v3.2
Parts:
- removed J4: ScreenIO, Connector_PinHeader_1.27mm:PinHeader_1x08_P1.27mm_Vertical
- removed R5: 10k, Resistor_SMD:R_0805_2012Metric
- removed U3: SHT4x, Sensor_Humidity:Sensirion_DFN-4_1.5x1.5mm_P0.8mm_SHT4x_NoCentralPad
- added R3: 10k, Resistor_SMD:R_0805_2012Metric, F.Cu at (89.0, 74.6)
- J1: footprint Connector_PinHeader_2.54mm:PinHeader_1x06_P2.54mm_Vertical -> Connector_PinHeader_1.27mm:PinHeader_1x10_P1.27mm_Vertical
- JP1, JP2: value 0x76 | 0x77 -> 0x76|0x77; footprint Jumper:SolderJumper-3_P2.0mm_Open_TrianglePad1.0x1.5mm -> Jumper:SolderJumper-3_P1.3mm_Open_RoundedPad1.0x1.5mm
- moved JP2 22.5 mm to (91.2, 70.1), turned to 90 degrees
- moved J3 17.6 mm to (74.8, 71.8)
- moved J2 17.3 mm to (71.9, 76.6)
- moved JP1 16.1 mm to (63.8, 52.9)
- moved U8 15.1 mm to (84.9, 70.2)
- moved J1 10.8 mm to (78.5, 78.1)
- moved U6 8.10 mm to (65.0, 60.0), turned to 180 degrees
- moved C6 5.87 mm to (62.0, 60.0)
- moved R2 3.82 mm to (68.4, 69.1)
- moved R1 3.66 mm to (72.8, 69.0)
- moved R4 3.63 mm to (85.0, 74.6), turned to 0 degrees
- moved H1 3.54 mm to (95.0, 45.0)
- moved H2 3.54 mm to (65.0, 45.0)
- moved H3 3.54 mm to (65.0, 75.0)
- moved H4 3.54 mm to (95.0, 75.0)
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Connections:
- J1 pad 1: +3V3 -> SDA
- J1 pad 2: GND -> SCL
- J1 pad 3: SDA -> 5V
- J1 pad 4: SCL -> GND
- J1 pad 5: SDA2 -> Tx
- J1 pad 6: SCL2 -> Rx
- R4 pad 2: SCL2 -> SDA2
Routing:
- net SDA: track 57.9 -> 34.5 mm, vias 1 -> 0
- net SCL: track 62.3 -> 39.4 mm
- net SDA2: track 36.7 -> 15.0 mm, vias 1 -> 0
- net SCL2: track 31.5 -> 16.3 mm
- net Rx: track 6.69 -> 16.4 mm
- net Tx: track 6.77 -> 16.4 mm
- net 5V: track 6.47 -> 15.8 mm
- net Net-(JP2-C): track 16.6 -> 8.22 mm, vias 0 -> 2
- net +3V3: track 30.8 -> 23.5 mm, vias 11 -> 4
- net Net-(JP1-C): track 2.44 -> 7.61 mm
- net GND: track 29.3 -> 24.1 mm, vias 9 -> 7
Other:
- board text added: "v3.2 - 2024.04.28 - niig"
- board text added: "v3.2 - 2024.04.29 - niig"
- board text removed: "3.3V"
- board text removed: "GND"
- board text removed: "SCL"
- board text removed: "SCL2"
- board text removed: "SDA"
- board text removed: "SDA2"
- board text removed: "v3.1 - 2024.04.27 - niig"

Commit message: complete airspeed v3.2
Other:
- board text added: "3V3"
- board text added: "5V"
- board text added: "GND"
- board text added: "Rx"
- board text added: "SCL"
- board text added: "SCL2"
- board text added: "SDA"
- board text added: "SDA2"
- board text added: "Tx"
Changed lines of the file:
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@@
     (fp_line (start 1 0.625) (end -1 0.625)
       (stroke (width 0.1) (type solid)) (layer "F.Fab"))
-    (pad "1" smd roundrect (at -0.9125 0 180) (size 1.025 1.4) (layers "F.Cu" "F.Paste" "F.Mask") (roundrect_rratio 0.243902)
+    (pad "1" smd roundrect (at -0.9125 0 180) (size 1.025 1.4) (layers "F.Cu" "F.Paste" "F.Mask") (roundrect_rratio 0.243902439)
       (net 18 "+3V3") (pintype "passive"))
-    (pad "2" smd roundrect (at 0.9125 0 180) (size 1.025 1.4) (layers "F.Cu" "F.Paste" "F.Mask") (roundrect_rratio 0.243902)
+    (pad "2" smd roundrect (at 0.9125 0 180) (size 1.025 1.4) (layers "F.Cu" "F.Paste" "F.Mask") (roundrect_rratio 0.243902439)
       (net 12 "SCL2") (pintype "passive"))
     (model "${KICAD6_3DMODEL_DIR}/Resistor_SMD.3dshapes/R_0805_2012Metric.wrl"
@@
     (fp_line (start 1 0.625) (end -1 0.625)
       (stroke (width 0.1) (type solid)) (layer "F.Fab"))
-    (pad "1" smd roundrect (at -0.9125 0) (size 1.025 1.4) (layers "F.Cu" "F.Paste" "F.Mask") (roundrect_rratio 0.243902)
+    (pad "1" smd roundrect (at -0.9125 0) (size 1.025 1.4) (layers "F.Cu" "F.Paste" "F.Mask") (roundrect_rratio 0.243902439)
       (net 18 "+3V3") (pintype "passive"))
-    (pad "2" smd roundrect (at 0.9125 0) (size 1.025 1.4) (layers "F.Cu" "F.Paste" "F.Mask") (roundrect_rratio 0.243902)
+    (pad "2" smd roundrect (at 0.9125 0) (size 1.025 1.4) (layers "F.Cu" "F.Paste" "F.Mask") (roundrect_rratio 0.243902439)
       (net 20 "SDA2") (pintype "passive"))
     (model "${KICAD6_3DMODEL_DIR}/Resistor_SMD.3dshapes/R_0805_2012Metric.wrl"
@@
         (effects (font (size 1 1) (thickness 0.15)) (justify mirror))
     )
-    (fp_text value "GPS" (at 0.1 -4.36) (layer "B.SilkS" knockout)
+    (fp_text value "GPS" (at -1.9 2.95) (layer "B.SilkS" knockout)
         (effects (font (size 1 1) (thickness 0.15)) (justify mirror))
     )
@@
         (effects (font (size 1 1) (thickness 0.15)) (justify mirror))
     )
-    (fp_text value "GPS" (at -6.6 2.6 180) (layer "B.SilkS" knockout)
+    (fp_text value "GPS" (at -0.2 -0.8 180) (layer "B.SilkS" knockout)
         (effects (font (size 1 1) (thickness 0.15)) (justify mirror))
     )
@@
     (effects (font (size 0.8 0.7) (thickness 0.125) bold) (justify left bottom mirror))
   )
+  (gr_text "SCL" (at 80.27 74.01 90) (layer "B.SilkS" knockout)
+    (effects (font (size 0.8 1) (thickness 0.1)) (justify left bottom mirror))
+  )
+  (gr_text "3V3" (at 90.38 74.08 90) (layer "B.SilkS" knockout)
+    (effects (font (size 0.8 1) (thickness 0.1)) (justify left bottom mirror))
+  )
+  (gr_text "Tx" (at 84.11 75.23 90) (layer "B.SilkS" knockout)
+    (effects (font (size 0.8 1) (thickness 0.1)) (justify left bottom mirror))
+  )
+  (gr_text "SCL2" (at 87.85 73.13 90) (layer "B.SilkS" knockout)
+    (effects (font (size 0.8 1) (thickness 0.1)) (justify left bottom mirror))
+  )
+  (gr_text "SDA" (at 79 73.96 90) (layer "B.SilkS" knockout)
+    (effects (font (size 0.8 1) (thickness 0.1)) (justify left bottom mirror))
+  )
+  (gr_text "Rx" (at 85.36 75 90) (layer "B.SilkS" knockout)
+    (effects (font (size 0.8 1) (thickness 0.1)) (justify left bottom mirror))
+  )
+  (gr_text "GND" (at 89.1 73.8 90) (layer "B.SilkS" knockout)
+    (effects (font (size 0.8 1) (thickness 0.1)) (justify left bottom mirror))
+  )
+  (gr_text "5V" (at 81.53 74.95 90) (layer "B.SilkS" knockout)
+    (effects (font (size 0.8 1) (thickness 0.1)) (justify left bottom mirror))
+  )
+  (gr_text "SDA2" (at 86.62 73.08 90) (layer "B.SilkS" knockout)
+    (effects (font (size 0.8 1) (thickness 0.1)) (justify left bottom mirror))
+  )
   (gr_text "velometa.com/airspeed" (at 88.8 43.4) (layer "B.SilkS" knockout)
     (effects (font (size 1 1) (thickness 0.15)) (justify left bottom mirror))
   )
+  (gr_text "GND" (at 82.86 73.8 90) (layer "B.SilkS" knockout)
+    (effects (font (size 0.8 1) (thickness 0.1)) (justify left bottom mirror))
+  )
   (gr_text "v3.2 - 2024.04.28 - niig" (at 71 44.9) (layer "F.SilkS")

Commit message: upgrade to kicad v8
Other:
- board text added: "${REVISION} - ${CURRENT_DATE} - niig"
- board text removed: "v3.2 - 2024.04.29 - niig"
