File: airspeed_v3/airspeed.kicad_pcb (KiCad board)
At the start: 2 copper layers, 40 x 40 mm, 20 parts, among them J1 Header, J2 GPS, J3 GPS, U1 XGZP6897D, U5 XGZP6897D, U6 BME280, U8 BMP280

Commit message: updated the schematic to use latest bp280
Parts:
- J2: value GPS -> GPS connector
- J3: value GPS -> GPS Header
Changed lines of the file:
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@@
 			)
 		)
-		(property "Description" ""
+		(property "Description" "Absolute Barometric Pressure Sensor, LGA-8"
 			(at 0 0 0)
 			(unlocked yes)
@@
 			)
 		)
+		(property ki_fp_filters "R_*")
+		(sheetname "Root")
+		(sheetfile "airspeed.kicad_sch")
 		(attr smd)
 		(fp_line
@@
 			)
 		)
+		(property ki_fp_filters "R_*")
+		(sheetname "Root")
+		(sheetfile "airspeed.kicad_sch")
 		(attr smd)
 		(fp_line
@@
 			)
 		)
+		(property ki_fp_filters "R_*")
+		(sheetname "Root")
+		(sheetfile "airspeed.kicad_sch")
 		(attr smd)
 		(fp_line
@@
 			)
 		)
-		(property "Value" "GPS"
+		(property "Value" "GPS Header"
 			(at -1.9 2.95 0)
 			(layer "B.SilkS" knockout)
@@
 			)
 		)
+		(property ki_fp_filters "R_*")
+		(sheetname "Root")
+		(sheetfile "airspeed.kicad_sch")
 		(attr smd)
 		(fp_line
@@
 		)
 		(property "Value" "XGZP6897D"
-			(at 0.16 -6.28 270)
+			(at 0.16 -6.28 -90)
 			(layer "F.SilkS" knockout)
 			(effects
@@
 		)
 		(property "Value" "XGZP6897D"
-			(at 0.03 6.22 270)
+			(at 0.03 6.22 -90)
 			(layer "F.SilkS" knockout)
 			(effects
@@
 			)
 		)
-		(property "Value" "GPS"
+		(property "Value" "GPS connector"
 			(at -0.2 -0.8 180)
 			(layer "B.SilkS")
@@
 			)
 		)
+		(property ki_fp_filters "Connector*:*_1x??_*")
+		(sheetname "Root")
+		(sheetfile "airspeed.kicad_sch")
 		(attr smd)
 		(fp_line
