File: airspeed_v3/airspeed.kicad_pcb (KiCad board)
At the start: 2 copper layers, 40 x 40 mm, 20 parts, among them J1 Header, J2 GPS connector, J3 GPS Header, U1 XGZP6897D, U5 XGZP6897D, U6 BME280, U8 BMP280

Commit message: v3.4
Parts:
- removed U5: XGZP6897D, niig:CFSensor_XGZP6897x
- removed U8: BMP280, Package_LGA:Bosch_LGA-8_2x2.5mm_P0.65mm_ClockwisePinNumbering
- added C10: 0.1pF, Capacitor_SMD:C_0805_2012Metric, F.Cu at (82.6, 72.5)
- added C2: 1uF, Capacitor_SMD:C_0805_2012Metric, F.Cu at (62.0, 59.9)
- added C3: 0.1pF, Capacitor_SMD:C_0805_2012Metric, F.Cu at (64.2, 57.0)
- added C9: 1uF, Capacitor_SMD:C_0805_2012Metric, F.Cu at (82.2, 67.1)
- added U2: XGZP6897D, Sensor_Pressure:CFSensor_XGZP6897x, F.Cu at (85.9, 60.0)
- added U3: BME280, Package_LGA:Bosch_LGA-8_2.5x2.5mm_P0.65mm_ClockwisePinNumbering, F.Cu at (84.9, 69.9)
- J2: value GPS connector -> GPS
- J3: value GPS Header -> GPS
- JP1, JP2: value 0x76|0x77 -> 0x77|0x76
- U1: footprint niig:CFSensor_XGZP6897x -> Sensor_Pressure:CFSensor_XGZP6897x
- moved C6 10.3 mm to (64.2, 70.0), turned to -90 degrees
- moved JP2 0.90 mm to (91.1, 69.2), turned to 0 degrees
- moved JP1 0.48 mm to (64.2, 52.7), turned to 0 degrees
Connections:
- JP2 pad 1: GND -> +3V3
- JP2 pad 3: +3V3 -> GND
Routing:
- net GND: track 24.1 -> 42.6 mm
- net +3V3: track 23.5 -> 31.2 mm
- net Net-(JP1-C): track 7.61 -> 6.36 mm
- net Net-(JP2-C): track 8.22 -> 9.07 mm
Other:
- board text added: "${REVISION} | ${CURRENT_DATE} | niig"
- board text removed: "${REVISION} - ${CURRENT_DATE} - niig"
- board text removed: "v3.2 - 2024.04.28 - niig"

Commit message: airspeed v3.6
Parts:
- added C11: 0.1uF, Capacitor_SMD:C_0805_2012Metric, F.Cu at (90.5, 75.8)
- added C12: 0.1pF, Capacitor_SMD:C_0805_2012Metric, F.Cu at (88.7, 67.9)
- added C13: 0.1uF, Capacitor_SMD:C_0805_2012Metric, F.Cu at (91.0, 71.0)
- added C14: 0.1uF, Capacitor_SMD:C_0805_2012Metric, F.Cu at (84.8, 75.4)
- added J4: Header, Connector_PinHeader_2.00mm:PinHeader_1x10_P2.00mm_Vertical, F.Cu at (69.0, 77.9)
- added J5: Header, Connector_PinHeader_1.27mm:PinHeader_1x10_P1.27mm_Vertical, F.Cu at (69.0, 73.4)
- added J6: Conn_01x04_Pin, Connector_PinHeader_1.27mm:PinHeader_1x04_P1.27mm_Vertical, F.Cu at (62.0, 67.0)
- added J7: Conn_01x04_Pin, Connector_PinHeader_1.27mm:PinHeader_1x04_P1.27mm_Vertical, F.Cu at (64.5, 67.0)
- added J8: Conn_01x04_Pin, Connector_PinHeader_1.27mm:PinHeader_1x04_P1.27mm_Vertical, F.Cu at (69.3, 60.4)
- added J9: Conn_01x07_Pin, Connector_Molex:Molex_PicoBlade_53047-0710_1x07_P1.25mm_Vertical, F.Cu at (98.1, 57.2)
- added U4: MPU-6050, Sensor_Motion:InvenSense_QFN-24_4x4mm_P0.5mm, F.Cu at (86.5, 71.6)
- J2: value GPS -> Conn_01x08_Pin; footprint Connector_JST:JST_SH_SM06B-SRSS-TB_1x06-1MP_P1.00mm_Horizontal -> Connector_Molex:Molex_PicoBlade_53047-0810_1x08_P1.25mm_Vertical; moved to F.Cu
- J3: value GPS -> GPS Header
- JP1: value 0x77|0x76 -> 0x76|0x77
- moved J2 27.0 mm to (98.1, 70.0), turned to 90 degrees
- moved C6 17.6 mm to (76.4, 57.4)
- moved J3 11.7 mm to (73.7, 60.1), turned to 0 degrees
- moved U2 10.8 mm to (85.8, 49.2)
- moved U1 10.8 mm to (73.9, 49.2)
- moved C5 10.8 mm to (76.1, 42.2)
- moved JP2 10.7 mm to (89.4, 58.6)
- moved C4 10.7 mm to (85.5, 42.2)
- moved J1 9.84 mm to (69.0, 75.4)
- moved C10 9.70 mm to (81.9, 62.8)
- moved C9 9.70 mm to (81.6, 57.4)
- moved U3 9.70 mm to (84.2, 60.2)
- moved R3 8.89 mm to (88.2, 65.8)
- moved R4 8.49 mm to (84.0, 66.2)
- moved C3 4.26 mm to (64.5, 52.8)
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Connections:
- J1 pad 5: Tx -> SCL3
- J1 pad 6: Rx -> SDA3
- J2 pad 1: Rx -> 5V
- J2 pad 2: Tx -> GND
- J2 pad 3: GND -> SDA
- J2 pad 4: 5V -> SCL
- J2 pad 5: SCL -> SDA2
- J2 pad 6: SDA -> SCL2
- J3 pad 1: Rx -> Tx
- J3 pad 2: Tx -> Rx
Routing:
- net SCL: track 39.4 -> 88.9 mm, vias 2 -> 0
- net SDA: track 34.5 -> 79.8 mm
- net SCL3: track 0.00 -> 40.4 mm, vias 0 -> 1
- net SDA3: track 0.00 -> 39.5 mm, vias 0 -> 1
- net SDA2: track 15.2 -> 52.5 mm, vias 0 -> 3
- net SCL2: track 16.3 -> 51.9 mm
- net 5V: track 15.8 -> 46.9 mm
- net Rx: track 16.4 -> 0.00 mm
- net GND: track 42.6 -> 57.9 mm, vias 7 -> 10
- net +3V3: track 31.2 -> 45.2 mm
- net Tx: track 16.4 -> 28.2 mm
- net Net-(U4-REGOUT): track 0.00 -> 4.10 mm
- net Net-(JP1-C): track 6.36 -> 4.50 mm
- net Net-(U4-CPOUT): track 0.00 -> 1.32 mm
Other:
- board text added: "Boot"
- board text added: "EN"
- board text added: "SCL3"
- board text added: "SDA3"
